File: schema/ledcube.brd (EAGLE design)
At the start: 100 x 50 mm, 64 parts, among them IC1 74LS595N, IC2 74LS595N, IC3 AVR-MEGA8-P, IC4 FT232RL-BASICSSOP, T1 BC547, T2 BC547, T3 BC547, T4 BC547, X1 USBSMD

Commit message: Schema bug updated
Parts:
- removed RXD, TXD: LSP10, solpad:LSP10
- added JP5: (no value), SparkFun:1X03
- moved C4 17.3 mm to (38.1, 24.1)
- moved C5 14.0 mm to (31.8, 46.4), turned to 0 degrees
- moved ISCP 1.80 mm to (27.3, 3.17), turned to 0 degrees
Connections:
- net +5V: now also IC1.10, IC2.10
- net GND: now also IC1.13, IC2.13, JP5.3
- net RXD: now also JP5.1; no longer RXD.MP
- net TXD: now also JP5.2; no longer TXD.MP
Routing:
- net RST: track 70.2 -> 80.7 mm
- net GND: track 40.7 -> 30.3 mm
- net N$57: track 28.3 -> 22.2 mm
- net MISO: track 29.9 -> 24.8 mm
- net N$11: track 15.7 -> 14.2 mm
- net SCK: track 24.8 -> 26.2 mm
- net MOSI: track 21.7 -> 20.6 mm
- net N$60: track 42.8 -> 43.7 mm
- net N$28: track 29.3 -> 29.9 mm
Other:
- board text added: "LedCube v1.2 20-12-2013 LeatiX"
- board text removed: "LedCube v1.1 13-05-2010 LeatiX"
