File: schema/ledcube.sch (EAGLE design)
At the start: 64 parts, among them IC1 74LS595N, IC2 74LS595N, IC3 AVR-MEGA8-P, IC4 FT232RL-BASICSSOP, T1 BC547, T2 BC547, T3 BC547, T4 BC547, X1 USBSMD

Commit message: Schema bug updated
Parts:
- removed RXD, TXD: LSP10, solpad:LSP10
- added JP5: (no value), SparkFun:M03PTH
Connections:
- net +5V: now also IC1.SCL, IC2.SCL
- net GND: now also IC1.G, IC2.G, JP5.3
- net RXD: now also JP5.1; no longer RXD.MP
- net TXD: now also JP5.2; no longer TXD.MP
Changed lines of the file:
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@@
 <part name="P+11" library="supply1" deviceset="+5V" device=""/>
 <part name="P+12" library="supply1" deviceset="+5V" device=""/>
-<part name="RXD" library="solpad" deviceset="LSP10" device=""/>
-<part name="TXD" library="solpad" deviceset="LSP10" device=""/>
+<part name="P+10" library="supply1" deviceset="+5V" device=""/>
+<part name="P+13" library="supply1" deviceset="+5V" device=""/>
+<part name="JP5" library="SparkFun" deviceset="M03" device="PTH"/>
+<part name="GND15" library="supply1" deviceset="GND" device=""/>
 </parts>
 <sheets>
@@
 <instance part="P+11" gate="1" x="83.82" y="-7.62"/>
 <instance part="P+12" gate="1" x="66.04" y="-7.62"/>
-<instance part="RXD" gate="1" x="71.12" y="81.28" rot="R270"/>
-<instance part="TXD" gate="1" x="68.58" y="78.74" rot="R270"/>
+<instance part="P+10" gate="1" x="119.38" y="78.74"/>
+<instance part="P+13" gate="1" x="116.84" y="17.78"/>
+<instance part="JP5" gate="G$1" x="76.2" y="78.74" rot="R180"/>
+<instance part="GND15" gate="1" x="66.04" y="71.12"/>
 </instances>
 <busses>
@@
 <wire x1="86.36" y1="-12.7" x2="83.82" y2="-12.7" width="0.1524" layer="91"/>
 <wire x1="83.82" y1="-12.7" x2="83.82" y2="-10.16" width="0.1524" layer="91"/>
+</segment>
+<segment>
+<pinref part="IC2" gate="A" pin="SCL"/>
+<wire x1="121.92" y1="66.04" x2="119.38" y2="66.04" width="0.1524" layer="91"/>
+<wire x1="119.38" y1="66.04" x2="119.38" y2="76.2" width="0.1524" layer="91"/>
+<pinref part="P+10" gate="1" pin="+5V"/>
+</segment>
+<segment>
+<pinref part="IC1" gate="A" pin="SCL"/>
+<pinref part="P+13" gate="1" pin="+5V"/>
+<wire x1="121.92" y1="7.62" x2="116.84" y2="7.62" width="0.1524" layer="91"/>
+<wire x1="116.84" y1="7.62" x2="116.84" y2="15.24" width="0.1524" layer="91"/>
 </segment>
 </net>
@@
 <pinref part="GND9" gate="1" pin="GND"/>
 <pinref part="IC2" gate="A" pin="GND"/>
+<wire x1="119.38" y1="50.8" x2="119.38" y2="55.88" width="0.1524" layer="91"/>
+<pinref part="IC2" gate="A" pin="G"/>
+<wire x1="119.38" y1="55.88" x2="121.92" y2="55.88" width="0.1524" layer="91"/>
 </segment>
 <segment>
@@
 <pinref part="GND8" gate="1" pin="GND"/>
 <pinref part="IC1" gate="A" pin="GND"/>
+<pinref part="IC1" gate="A" pin="G"/>
+<wire x1="121.92" y1="-2.54" x2="119.38" y2="-2.54" width="0.1524" layer="91"/>
+<wire x1="119.38" y1="-2.54" x2="119.38" y2="-7.62" width="0.1524" layer="91"/>
 </segment>
 <segment>
@@
 <wire x1="73.66" y1="27.94" x2="73.66" y2="25.4" width="0.1524" layer="91"/>
 <pinref part="JP1" gate="G$1" pin="2"/>
+</segment>
+<segment>
+<pinref part="JP5" gate="G$1" pin="3"/>
+<pinref part="GND15" gate="1" pin="GND"/>
+<wire x1="68.58" y1="76.2" x2="66.04" y2="76.2" width="0.1524" layer="91"/>
+<wire x1="66.04" y1="76.2" x2="66.04" y2="73.66" width="0.1524" layer="91"/>
 </segment>
 </net>
@@
 </segment>
 <segment>
-<pinref part="TXD" gate="1" pin="MP"/>
-<wire x1="66.04" y1="78.74" x2="58.42" y2="78.74" width="0.1524" layer="91"/>
+<wire x1="68.58" y1="78.74" x2="58.42" y2="78.74" width="0.1524" layer="91"/>
 <label x="58.42" y="78.74" size="1.778" layer="95"/>
+<pinref part="JP5" gate="G$1" pin="2"/>
 </segment>
 </net>
@@
 </segment>
 <segment>
-<pinref part="RXD" gate="1" pin="MP"/>
 <wire x1="68.58" y1="81.28" x2="58.42" y2="81.28" width="0.1524" layer="91"/>
 <label x="58.42" y="81.28" size="1.778" layer="95"/>
-</segment>
-</net>
+<pinref part="JP5" gate="G$1" pin="1"/>
+</segment>
+</net>
